File: Hardware/BreakoutBoard_STM32F411/HMI_Debbug.kicad_sch (KiCad schematic)
At the start: 4 parts

Commit message: routed PCB (#4)
Parts:
- D301: value LED -> 3.3V
- D302: value LED -> 5V
Other:
- moved on the sheet: D301
Changed lines of the file:
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@@
 	(symbol
 		(lib_id "Device:LED")
-		(at 59.69 71.12 90)
-		(unit 1)
-		(exclude_from_sim no)
-		(in_bom yes)
-		(on_board yes)
-		(dnp no)
-		(fields_autoplaced yes)
+		(at 59.69 71.12 270)
+		(mirror x)
+		(unit 1)
+		(exclude_from_sim no)
+		(in_bom yes)
+		(on_board yes)
+		(dnp no)
 		(property "Reference" "D301"
-			(at 57.15 73.9776 90)
-			(effects
-				(font
-					(size 1.27 1.27)
-				)
-				(justify left)
-			)
-		)
-		(property "Value" "LED"
-			(at 57.15 71.4376 90)
-			(effects
-				(font
-					(size 1.27 1.27)
-				)
-				(justify left)
+			(at 55.88 71.4374 90)
+			(effects
+				(font
+					(size 1.27 1.27)
+				)
+				(justify right)
+			)
+		)
+		(property "Value" "3.3V"
+			(at 55.88 73.9774 90)
+			(effects
+				(font
+					(size 1.27 1.27)
+				)
+				(justify right)
 			)
 		)
@@
 		(fields_autoplaced yes)
 		(property "Reference" "D302"
-			(at 69.85 73.9776 90)
-			(effects
-				(font
-					(size 1.27 1.27)
-				)
-				(justify left)
-			)
-		)
-		(property "Value" "LED"
-			(at 69.85 71.4376 90)
-			(effects
-				(font
-					(size 1.27 1.27)
-				)
-				(justify left)
-			)
-		)
+			(at 76.2 71.4374 90)
+			(effects
+				(font
+					(size 1.27 1.27)
+				)
+				(justify right)
+			)
+		)
+		(property "Value" "5V"
+			(at 76.2 73.9774 90)
+			(effects
+				(font
+					(size 1.27 1.27)
+				)
+				(justify right)
+			)
+		)
