File: Hardware/BreakoutBoard_STM32F411/BreakoutBoard_STM32F411.kicad_sch (KiCad schematic)
At the start: 0 parts

Commit message: added:components (#1)
Parts:
- added C101: 1uF, Capacitor_SMD:C_0603_1608Metric, symbol Device:C
- added C102, C103, C104, C106, C107: 100nF, Capacitor_SMD:C_0402_1005Metric, symbol Device:C
- added C105: 4.7uF, Capacitor_SMD:C_0805_2012Metric, symbol Device:C
- added IC101: STM32F411CCU6TR, SamacSys_Parts:QFN50P700X700X65-49N-D, symbol SamacSys_Parts:STM32F411CCU6TR
- added Y101: ASDDV-16.000MHZ-LR-T, SamacSys_Parts:AbraconASDDV, symbol SamacSys_Parts:ASDDV-16.000MHZ-LR-T
Connections:
- new net: C105.2, IC101.22 (VCAP_1)
- new net +3.3V: C101.2, C102.1, C103.2, C104.1, C106.1, C107.1, IC101.24 (VDD_1), IC101.36 (VDD_2), IC101.48 (VDD_3), IC101.9 (VDDA/VREF+), Y101.4 (VDD)
- new net GND: C101.1, C102.2, C103.1, C104.2, C105.1, C106.2, C107.2, IC101.23 (VSS_1), IC101.35 (VSS_2), IC101.47 (VSS_3), IC101.49 (GND), IC101.8 (VSSA/VREF_-), Y101.2 (GND)
- new net PA0: IC101.10 (PA0)
- new net PA1: IC101.11 (PA1)
- new net PA10: IC101.31 (PA10)
- new net PA11: IC101.32 (PA11)
- new net PA12: IC101.33 (PA12)
- new net PA13 | SYS_SWDIO: IC101.34 (PA13)
- new net PA14 | SYS_SWCLK: IC101.37 (PA14)
- new net PA15 | TIM2_CH1: IC101.38 (PA15)
- new net PA2: IC101.12 (PA2)
- new net PA3: IC101.13 (PA3)
- new net PA4: IC101.14 (PA4)
- new net PA5: IC101.15 (PA5)
- new net PA6: IC101.16 (PA6)
- new net PA7: IC101.17 (PA7)
- new net PA8: IC101.29 (PA8)
- new net PA9: IC101.30 (PA9)
- new net PB0: IC101.18 (PB0)
- new net PB1: IC101.19 (PB1)
- new net PB10 | I2C2_SCL: IC101.21 (PB10)
- new net PB12: IC101.25 (PB12)
- new net PB13 | SPI2_SCK: IC101.26 (PB13)
- new net PB14 | SPI2_MISO: IC101.27 (PB14)
- new net PB15 | SPI2_MOSI: IC101.28 (PB15)
- new net PB2: IC101.20 (PB2)
- new net PB3: IC101.39 (PB3)
- new net PB4: IC101.40 (PB4)
- new net PB5: IC101.41 (PB5)
- new net PB6: IC101.42 (PB6)
- new net PB7: IC101.43 (PB7)
- new net PB8: IC101.45 (PB8)
- new net PB9 | I2C2_SDA: IC101.46 (PB9)
- new net PH0: IC101.5 (PH0-OSC_IN), Y101.3 (OUTPUT)
Other:
- added sheet HMI_Debbug_4 (HMI_Debbug.kicad_sch)
- added sheet Power_3 (Power.kicad_sch)
- added sheet connectivity_2 (connectivity.kicad_sch)

Commit message: fixed:Viasize, fixed:NRST and BOOT0 (#5)
Parts:
- added C405: 100nF, Capacitor_SMD:C_0402_1005Metric, symbol Device:C
- added R401, R402: 10k, Resistor_SMD:R_0402_1005Metric, symbol Device:R
Connections:
- net +3.3V: now also R401.1
- net GND: now also C405.2, R402.2
- net BOOT0: now reaches IC101.44 (BOOT0)
- net BOOT0: now also R401.2, R402.1
- net NRST: now reaches IC101.7 (NRST)
- net NRST: now also C405.1

Commit message: ordering Version
Parts:
- C103: value 100nF -> 10nF
Changed lines of the file:
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@@
 			)
 		)
-		(property "Value" "100nF"
+		(property "Value" "10nF"
 			(at 39.116 172.974 90)
 			(effects
